File: Multi AV QSB/MultiOut.kicad_sch (KiCad schematic)
At the start: 2 parts, among them J1 RGB_OUT, J2 Multi AV

Commit message: Prepping for release
Other:
- company: (none) -> ThunderTechnologies
- title: (none) -> MultOut QSB
Changed lines of the file:
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@@
 	(generator_version "8.0")
 	(paper "A4")
+	(title_block
+		(title "MultOut QSB")
+		(date "2024-08-31")
+		(rev "1")
+		(company "ThunderTechnologies")
+		(comment 1 "Designed by InnocuousMuffin")
+	)
 	(junction
 		(at 175.26 58.42)
