File: SNEdge PCB - rev2/SNEdge.kicad_pcb (KiCad board)
At the start: 2 copper layers, 40.8 x 18.4 mm, 33 parts, among them J10 R_O, J8 G_O, J9 B_O, U1 THS7376

Commit message: Small SNEdge update for THS VCC decoupling cap
Parts:
- moved C2 1.40 mm to (112.8, 106.0)
Routing:
- net VCC: track 40.4 -> 37.6 mm
- net GND: vias 44 -> 43
Changed lines of the file:
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@@
 				(font
 					(size 0.7 0.7)
-					(thickness 0.15)
+					(thickness 0.175)
 				)
 			)
@@
 	(footprint "Capacitor_SMD:C_0805_2012Metric_Pad1.18x1.45mm_HandSolder"
 		(layer "F.Cu")
-		(at 111.4 106)
+		(at 112.8 106)
 		(descr "Capacitor SMD 0805 (2012 Metric), square (rectangular) end terminal, IPC-7351 nominal with elongated pad for handsoldering. (Body size source: IPC-SM-782 page 76, https://www.pcb-3d.com/wordpress/wp-content/uploads/ipc-sm-782a_amendment_1_and_2.pdf, https://docs.google.com/spreadsheets/d/1BsfQQcO9C6DZCsRaXUlFlo91Tg2WpOkGARC1WS5S8t0/edit?usp=sharing), generated with kicad-footprint-generator")
 		(tags "capacitor handsolder")
@@
 			(effects
 				(font
-					(size 0.6 0.6)
-					(thickness 0.15)
+					(size 0.7 0.7)
+					(thickness 0.175)
 				)
 			)
@@
 				(font
 					(size 0.7 0.7)
-					(thickness 0.15)
+					(thickness 0.175)
 				)
 			)
@@
 				(font
 					(size 0.7 0.7)
-					(thickness 0.15)
+					(thickness 0.175)
 				)
 			)
@@
 	)
 	(segment
+		(start 114 106)
+		(end 115.35 104.65)
+		(width 0.2)
+		(layer "F.Cu")
+		(net 1)
+	)
+	(segment
 		(start 142.7 98.2)
 		(end 142.7 98.1)
@@
 	)
 	(segment
-		(start 112.4375 106)
-		(end 112.46987 106)
-		(width 0.2)
-		(layer "F.Cu")
-		(net 1)
-	)
-	(segment
 		(start 139.2 96.9)
 		(end 138.1625 97.9375)
@@
 	)
 	(segment
-		(start 114 106)
-		(end 115.35 104.65)
-		(width 0.2)
-		(layer "F.Cu")
-		(net 1)
-	)
-	(segment
-		(start 112.46987 106)
+		(start 113.8375 106)
 		(end 114 106)
 		(width 0.2)
@@
 	)
 	(via
-		(at 112.46987 106)
+		(at 113.86987 106)
 		(size 0.6)
 		(drill 0.3)
@@
 	)
 	(segment
-		(start 122.9 106)
-		(end 112.46987 106)
+		(start 138.1625 98.2)
+		(end 130.7 98.2)
 		(width 0.3)
 		(layer "B.Cu")
@@
 	)
 	(segment
-		(start 138.1625 98.2)
-		(end 130.7 98.2)
+		(start 122.9 106)
+		(end 113.86987 106)
 		(width 0.3)
 		(layer "B.Cu")
@@
 		(size 0.6)
 		(drill 0.3)
-		(layers "F.Cu" "B.Cu")
-		(free yes)
-		(net 2)
-	)
-	(via
-		(at 113.7 105.1)
-		(size 0.6)
-		(drill 0.3)

Commit message: Update references and a bit of clean up
Parts:
- C3, C4, C5: value 27pF -> 15pF
- R1, R2, R3: value 10k -> 7.5k
- moved C1 25.5 mm to (164.7, 98.0)
- moved FB1 25.5 mm to (169.2, 98.0)
- moved J8 25.5 mm to (159.2, 93.2)
- moved C2 25.5 mm to (138.3, 105.8)
- moved C6 25.5 mm to (133.7, 96.7)
- moved R10 25.5 mm to (137.7, 101.6)
- moved R2 25.5 mm to (142.3, 93.0)
- moved R3 25.5 mm to (147.3, 93.0)
- moved R4 25.5 mm to (135.7, 101.6)
- moved R7 25.5 mm to (133.7, 101.6)
- moved TP3 25.5 mm to (147.3, 92.0)
- moved TP4 25.5 mm to (142.3, 92.0)
- moved TP6 25.5 mm to (136.7, 96.8)
- moved TP7 25.5 mm to (146.7, 96.8)
- moved C3 25.5 mm to (140.2, 99.4)
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- renumbered R12 to R11, R11 to R12, R5 to R4, R7 to R5, R9 to R6, R4 to R7, R6 to R8, R8 to R9
