File: SNEdge PCB - rev2/SNEdge.kicad_sch (KiCad schematic)
At the start: 33 parts, among them J10 R_O, J8 G_O, J9 B_O, U1 THS7376

Commit message: Update references and a bit of clean up
Parts:
- C3, C4, C5: value 27pF -> 15pF
- R1, R2, R3: value 10k -> 7.5k
- renumbered R12 to R11, R11 to R12, R5 to R4, R7 to R5, R9 to R6, R4 to R7, R6 to R8, R8 to R9
Changed lines of the file:
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@@
 		(on_board yes)
 		(dnp no)
-		(property "Reference" "R8"
+		(property "Reference" "R9"
 			(at 170.942 54.102 90)
 			(effects
@@
 			(project "SNEdge"
 				(path "/b6c15655-575b-4e1d-9394-554f8b7e5fea"
-					(reference "R8")
+					(reference "R9")
 					(unit 1)
 				)
@@
 		(on_board yes)
 		(dnp no)
-		(property "Reference" "R6"
+		(property "Reference" "R8"
 			(at 149.86 53.848 90)
 			(effects
@@
 			(project "SNEdge"
 				(path "/b6c15655-575b-4e1d-9394-554f8b7e5fea"
-					(reference "R6")
+					(reference "R8")
 					(unit 1)
 				)
@@
 			)
 		)
-		(property "Value" "10k"
+		(property "Value" "7.5k"
 			(at 108.204 127.254 0)
 			(effects
@@
 		(on_board yes)
 		(dnp no)
-		(property "Reference" "R12"
+		(property "Reference" "R11"
 			(at 175.768 106.934 90)
 			(effects
@@
 			(project "SNEdge"
 				(path "/b6c15655-575b-4e1d-9394-554f8b7e5fea"
-					(reference "R12")
+					(reference "R11")
 					(unit 1)
 				)
@@
 		(on_board yes)
 		(dnp no)
-		(property "Reference" "R7"
+		(property "Reference" "R5"
 			(at 159.766 64.77 0)
 			(effects
@@
 			(project "SNEdge"
 				(path "/b6c15655-575b-4e1d-9394-554f8b7e5fea"
-					(reference "R7")
+					(reference "R5")
 					(unit 1)
 				)
@@
 		(on_board yes)
 		(dnp no)
-		(property "Reference" "R5"
+		(property "Reference" "R4"
 			(at 139.7 64.77 0)
 			(effects
@@
 			(project "SNEdge"
 				(path "/b6c15655-575b-4e1d-9394-554f8b7e5fea"
-					(reference "R5")
+					(reference "R4")
 					(unit 1)
 				)
@@
 			)
 		)
-		(property "Value" "10k"
+		(property "Value" "7.5k"
 			(at 108.204 109.474 0)
 			(effects
@@
 			)
 		)
-		(property "Value" "27pF"
+		(property "Value" "15pF"
 			(at 141.478 90.424 90)
 			(effects
@@
 		(on_board yes)
 		(dnp no)
-		(property "Reference" "R9"
+		(property "Reference" "R6"
 			(at 181.864 64.516 0)
 			(effects
@@
 			(project "SNEdge"
 				(path "/b6c15655-575b-4e1d-9394-554f8b7e5fea"
-					(reference "R9")
+					(reference "R6")
 					(unit 1)
 				)
@@
 			)
 		)
-		(property "Value" "27pF"
+		(property "Value" "15pF"
 			(at 141.732 77.47 90)
 			(effects
@@
 			)
 		)
-		(property "Value" "10k"
+		(property "Value" "7.5k"
 			(at 108.204 92.964 0)
 			(effects
@@
 			)
 		)
-		(property "Value" "27pF"
+		(property "Value" "15pF"
 			(at 141.986 84.074 90)
 			(effects
@@
 		(on_board yes)
 		(dnp no)
-		(property "Reference" "R4"
+		(property "Reference" "R7"
 			(at 129.286 53.848 90)
 			(effects
@@
 			(project "SNEdge"
 				(path "/b6c15655-575b-4e1d-9394-554f8b7e5fea"
-					(reference "R4")
+					(reference "R7")
 					(unit 1)
 				)
@@
 		(on_board yes)
 		(dnp no)
-		(property "Reference" "R11"
+		(property "Reference" "R12"
 			(at 175.768 104.394 90)
 			(effects
@@
 			(project "SNEdge"
 				(path "/b6c15655-575b-4e1d-9394-554f8b7e5fea"
-					(reference "R11")
+					(reference "R12")
 					(unit 1)
 				)
