File: SNEdge PCB/SNEdge.kicad_sch (KiCad schematic)
At the start: 40 parts, among them J1 RGB_OUT, U1 THS7376

Commit message: Updating the branch to include all stuff from collab
Parts:
- removed C3, C5: 3pF, Capacitor_SMD:C_0805_2012Metric, symbol Device:C_Small
- removed C7: 100nF, Capacitor_SMD:C_0805_2012Metric, symbol Device:C_Small
- removed JP1, JP2, JP3: SIDECAR, Jumper:SolderJumper-2_P1.3mm_Open_RoundedPad1.0x1.5mm, symbol Jumper:SolderJumper_2_Open
- removed TP10: G_OUT, TestPoint:TestPoint_Pad_1.0x1.0mm, symbol Connector:TestPoint
- removed TP11: B_OUT, TestPoint:TestPoint_Pad_1.0x1.0mm, symbol Connector:TestPoint
- removed TP12: G_ENC, TestPoint:TestPoint_Pad_2.0x2.0mm, symbol Connector:TestPoint
- removed TP13: B_ENC, TestPoint:TestPoint_Pad_2.0x2.0mm, symbol Connector:TestPoint
- removed TP14: R_ENC, TestPoint:TestPoint_Pad_2.0x2.0mm, symbol Connector:TestPoint
- removed TP15: GND, TestPoint:TestPoint_Pad_2.0x2.0mm, symbol Connector:TestPoint
- removed TP16: GND, TestPoint:TestPoint_Pad_1.0x1.0mm, symbol Connector:TestPoint
- removed TP9: R_OUT, TestPoint:TestPoint_Pad_1.0x1.0mm, symbol Connector:TestPoint
- added C2: 1uF, Capacitor_SMD:C_0805_2012Metric_Pad1.18x1.45mm_HandSolder, symbol Device:C_Small
- added J10: R_O, Connector_Coaxial:U.FL_Hirose_U.FL-R-SMT-1_Vertical, symbol Connector:Conn_Coaxial_Small
- added J8: G_O, Connector_Coaxial:U.FL_Hirose_U.FL-R-SMT-1_Vertical, symbol Connector:Conn_Coaxial_Small
- added J9: B_O, Connector_Coaxial:U.FL_Hirose_U.FL-R-SMT-1_Vertical, symbol Connector:Conn_Coaxial_Small
- added JP1: INPUT JUMPER, TT_Jumpers:R_0805_2012Metric_Pad1.20x1.40mm_HandSolder_Jumper_Closed, symbol Jumper:SolderJumper_2_Bridged
- added R1, R2, R3: 7.5k, Resistor_SMD:R_0805_2012Metric_Pad1.20x1.40mm_HandSolder, symbol Device:R_US
- added R13, R14, R15: 110R, Resistor_SMD:R_0805_2012Metric_Pad1.20x1.40mm_HandSolder, symbol Device:R_US
- C1: value 3pF -> 22uF; footprint Capacitor_SMD:C_0805_2012Metric -> Capacitor_SMD:C_0805_2012Metric_Pad1.18x1.45mm_HandSolder; Digi_PN 311-1092-1-ND -> 490-GRM21BZ71A226ME15KCT-ND; MFG_PN CC0805CRNPO9BN3R0 -> GRM21BZ71A226ME15K
- C3: renamed from C2; value 24pF -> 10pF; footprint Capacitor_SMD:C_0805_2012Metric -> Capacitor_SMD:C_0805_2012Metric_Pad1.18x1.45mm_HandSolder; Digi_PN 478-10387-1-ND -> 478-KGM21BCG1H100FTCT-ND; MFG_PN 08051A240FAT2A -> KGM21BCG1H100FT; Tolerance (none) -> 1%
- C4: value 24pF -> 10pF; footprint Capacitor_SMD:C_0805_2012Metric -> Capacitor_SMD:C_0805_2012Metric_Pad1.18x1.45mm_HandSolder; Digi_PN 478-10387-1-ND -> 478-KGM21BCG1H100FTCT-ND; MFG_PN 08051A240FAT2A -> KGM21BCG1H100FT; Tolerance (none) -> 1%
- C5: renamed from C6; value 24pF -> 10pF; footprint Capacitor_SMD:C_0805_2012Metric -> Capacitor_SMD:C_0805_2012Metric_Pad1.18x1.45mm_HandSolder; Digi_PN 478-10387-1-ND -> 478-KGM21BCG1H100FTCT-ND; MFG_PN 08051A240FAT2A -> KGM21BCG1H100FT; Tolerance (none) -> 1%
- C6: renamed from C10; value 100nF -> 1uF; footprint Capacitor_SMD:C_0805_2012Metric -> Capacitor_SMD:C_0805_2012Metric_Pad1.18x1.45mm_HandSolder; Digi_PN 1276-2444-1-ND -> 1276-1029-1-ND; MFG_PN CL21B104KBCNFNC -> CL21B105KBFNNNE
- C7: renamed from C9; value 100nF -> 1uF; footprint Capacitor_SMD:C_0805_2012Metric -> Capacitor_SMD:C_0805_2012Metric_Pad1.18x1.45mm_HandSolder; Digi_PN 1276-2444-1-ND -> 1276-1029-1-ND; MFG_PN CL21B104KBCNFNC -> CL21B105KBFNNNE
- C8: value 100nF -> 1uF; footprint Capacitor_SMD:C_0805_2012Metric -> Capacitor_SMD:C_0805_2012Metric_Pad1.18x1.45mm_HandSolder; Digi_PN 1276-2444-1-ND -> 1276-1029-1-ND; MFG_PN CL21B104KBCNFNC -> CL21B105KBFNNNE
- R10: renamed from R7; value 510R -> 240R; footprint Resistor_SMD:R_0805_2012Metric -> Resistor_SMD:R_0805_2012Metric_Pad1.20x1.40mm_HandSolder; Digi_PN RMCF0805FT510RCT-ND -> RMCF0805FT240RCT-ND; MFG_PN RMCF0805FT510R -> RMCF0805FT240R; Tolerance (none) -> 1%
- R11: renamed from R6; value 510R -> 240R; footprint Resistor_SMD:R_0805_2012Metric -> Resistor_SMD:R_0805_2012Metric_Pad1.20x1.40mm_HandSolder; Digi_PN RMCF0805FT510RCT-ND -> RMCF0805FT240RCT-ND; MFG_PN RMCF0805FT510R -> RMCF0805FT240R; Tolerance (none) -> 1%
- R12: renamed from R5; value 510R -> 240R; footprint Resistor_SMD:R_0805_2012Metric -> Resistor_SMD:R_0805_2012Metric_Pad1.20x1.40mm_HandSolder; Digi_PN RMCF0805FT510RCT-ND -> RMCF0805FT240RCT-ND; MFG_PN RMCF0805FT510R -> RMCF0805FT240R; Tolerance (none) -> 1%
- R4: renamed from R8; value 1k -> 430R; footprint Resistor_SMD:R_0805_2012Metric -> Resistor_SMD:R_0805_2012Metric_Pad1.20x1.40mm_HandSolder; Digi_PN RMCF0805FT1K00CT-ND -> 311-430CRCT-ND; MFG_PN RMCF0805FT1K00 -> RC0805FR-07430RL; Tolerance (none) -> 1%
- R5: renamed from R3; value 1k -> 430R; footprint Resistor_SMD:R_0805_2012Metric -> Resistor_SMD:R_0805_2012Metric_Pad1.20x1.40mm_HandSolder; Digi_PN RMCF0805FT1K00CT-ND -> 311-430CRCT-ND; MFG_PN RMCF0805FT1K00 -> RC0805FR-07430RL; Tolerance (none) -> 1%
- R6: renamed from R1; value 1k -> 430R; footprint Resistor_SMD:R_0805_2012Metric -> Resistor_SMD:R_0805_2012Metric_Pad1.20x1.40mm_HandSolder; Digi_PN RMCF0805FT1K00CT-ND -> 311-430CRCT-ND; MFG_PN RMCF0805FT1K00 -> RC0805FR-07430RL; Tolerance (none) -> 1%
- R7: renamed from R9; value 150R -> 75R; footprint Resistor_SMD:R_0805_2012Metric -> Resistor_SMD:R_0805_2012Metric_Pad1.20x1.40mm_HandSolder; Digi_PN RMCF0805FT150RCT-ND -> RNCP0805FTD75R0CT-ND; MFG_PN RMCF0805FT150R -> RNCP0805FTD75R0; Tolerance (none) -> 1%
- R8: renamed from R4; value 150R -> 75R; footprint Resistor_SMD:R_0805_2012Metric -> Resistor_SMD:R_0805_2012Metric_Pad1.20x1.40mm_HandSolder; Digi_PN RMCF0805FT150RCT-ND -> RNCP0805FTD75R0CT-ND; MFG_PN RMCF0805FT150R -> RNCP0805FTD75R0; Tolerance (none) -> 1%
- R9: renamed from R2; value 150R -> 75R; footprint Resistor_SMD:R_0805_2012Metric -> Resistor_SMD:R_0805_2012Metric_Pad1.20x1.40mm_HandSolder; Digi_PN RMCF0805FT150RCT-ND -> RNCP0805FTD75R0CT-ND; MFG_PN RMCF0805FT150R -> RNCP0805FTD75R0; Tolerance (none) -> 1%
- TP1, TP2, TP5: footprint TestPoint:TestPoint_Pad_2.0x2.0mm -> TestPoint:TestPoint_Pad_1.5x1.5mm
- TP3: value GND -> G_IN; footprint TestPoint:TestPoint_Pad_2.0x2.0mm -> TestPoint:TestPoint_Pad_1.5x1.5mm
- TP4: value GND -> B_IN; footprint TestPoint:TestPoint_Pad_2.0x2.0mm -> TestPoint:TestPoint_Pad_1.5x1.5mm
- TP6: value G_IN -> R_E; footprint TestPoint:TestPoint_Pad_2.0x2.0mm -> TestPoint:TestPoint_Pad_1.5x1.5mm
- TP7: value B_IN -> B_E; footprint TestPoint:TestPoint_Pad_2.0x2.0mm -> TestPoint:TestPoint_Pad_1.5x1.5mm
- TP8: value GND -> G_E; footprint TestPoint:TestPoint_Pad_2.0x2.0mm -> TestPoint:TestPoint_Pad_1.5x1.5mm
Connections:
- net GND: now also C1.1, U1.9 (BYPASS), C2.1, J10.2 (Ext), J8.2 (Ext), J9.2 (Ext), R1.1, R13.2, R14.2, R15.2, R2.1, R3.1; no longer TP3.1, TP4.1, TP8.1
- net VCC: now also C1.2, C2.2, JP1.2 (B); no longer TP1.1, U1.9 (BYPASS)
- net at C6.2: now also TP6.1
- net at C3.1, R10.2, U1.11 (CH4_OUT): now also R4.1; no longer R5.1
- net at C4.1, R11.2, U1.12 (CH3_OUT): now also R5.1; no longer R6.1
- net at C5.1, R12.2, U1.13 (CH2_OUT): now also R6.1; no longer R4.1
- net at C5.2, U1.2 (CH2_IN): now also TP3.1, R3.2; no longer TP5.1
- net at C4.2, U1.3 (CH3_IN): now also TP4.1, R2.2; no longer TP6.1
- net at C3.2, U1.4 (CH4_IN): now also TP5.1, R1.2; no longer C1.2, TP7.1
- net at R10.1: now also J1.6 (Pin_6), J10.1 (In), R15.1; no longer J1.2 (Pin_2)
- net at J1.4 (Pin_4): now also R12.1, J8.1 (In), R13.1; no longer R11.1
- net at C7.2: now also TP7.1
- net at C8.2: now also TP8.1
- new net: J1.2 (Pin_2), J9.1 (In), R11.1, R14.1
- new net: JP1.1 (A), TP1.1
Other:
- company: Thunder Technologies -> Innov8bit And ThunderTechnologies
- moved on the sheet: C3, C4, C5, C6, C7, C8, J1, R10, R11, R12, R4, R5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
